File: KiCAD/usbasp.sch (KiCad schematic (older format))
At the start: 21 parts, among them IC1 ATMEGA88-A, P1 ISP, P2 SelfPrograming, P2 VoltageSelect, P3 SlowCLK, P3 USB_B, U1 AP1117

Commit message: PCB layout WiP
Parts:
- 12MHz1: renamed from 12MHz; footprint (none) -> Crystals:Crystal_HC49-U_Vertical
- 22pF1, 22pF2: renamed from 22pF; footprint (none) -> Capacitors_SMD:C_0805_HandSoldering
- D3, D4: footprint (none) -> LEDs:LED-5MM
- D5, D6: renamed from D1; footprint (none) -> Diodes_ThroughHole:Diode_DO-35_SOD27_Horizontal_RM10
- IC1: footprint TQFP32 -> Housings_QFP:TQFP-32_7x7mm_Pitch0.8mm
- P1: footprint (none) -> Pin_Headers:Pin_Header_Angled_2x05
- P2: footprint (none) -> Pin_Headers:Pin_Header_Angled_1x03
- P3: footprint (none) -> Pin_Headers:Pin_Header_Angled_1x02
- P4: renamed from P2; footprint (none) -> Pin_Headers:Pin_Header_Angled_1x02
- P5: renamed from P3; footprint (none) -> Connect:USB_A
- R1, R10, R2, R5, R9: footprint (none) -> Resistors_SMD:R_0805
- R11, R8: footprint (none) -> Resistors_SMD:R_0805_HandSoldering
- U1: footprint (none) -> SMD_Packages:SOT-223
Changed lines of the file:
@@
 F 0 "IC1" H 900 7550 40  0000 L BNN
 F 1 "ATMEGA88-A" H 2100 4900 40  0000 L BNN
-F 2 "TQFP32" H 1650 6300 30  0000 C CIN
+F 2 "Housings_QFP:TQFP-32_7x7mm_Pitch0.8mm" H 1650 6300 30  0001 C CIN
 F 3 "" H 1650 6300 60  0000 C CNN
 	1    1650 6300
@@
 TXD
 $Comp
-L VCC #PWR?
+L VCC #PWR01
 U 1 1 55BF17CC
 P 600 5100
-F 0 "#PWR?" H 600 4950 50  0001 C CNN
+F 0 "#PWR01" H 600 4950 50  0001 C CNN
 F 1 "VCC" H 600 5250 50  0000 C CNN
 F 2 "" H 600 5100 60  0000 C CNN
@@
 Connection ~ 600  5500
 $Comp
-L GND #PWR?
+L GND #PWR02
 U 1 1 55BF1808
 P 550 7600
-F 0 "#PWR?" H 550 7350 50  0001 C CNN
+F 0 "#PWR02" H 550 7350 50  0001 C CNN
 F 1 "GND" H 550 7450 50  0000 C CNN
 F 2 "" H 550 7600 60  0000 C CNN
@@
 Connection ~ 550  7500
 $Comp
-L Crystal 12MHz
+L Crystal 12MHz1
 U 1 1 55BF186C
 P 3950 4900
-F 0 "12MHz" H 3950 5050 50  0000 C CNN
+F 0 "12MHz1" H 3950 5050 50  0000 C CNN
 F 1 "Crystal" H 3950 4750 50  0000 C CNN
-F 2 "" H 3950 4900 60  0000 C CNN
+F 2 "Crystals:Crystal_HC49-U_Vertical" H 3950 4900 60  0001 C CNN
 F 3 "" H 3950 4900 60  0000 C CNN
 	1    3950 4900
@@
 $EndComp
 $Comp
-L C 22pF
+L C 22pF1
 U 1 1 55BF1990
 P 4350 4750
-F 0 "22pF" H 4375 4850 50  0000 L CNN
+F 0 "22pF1" H 4375 4850 50  0000 L CNN
 F 1 "C1" H 4375 4650 50  0000 L CNN
-F 2 "" H 4388 4600 30  0000 C CNN
+F 2 "Capacitors_SMD:C_0805_HandSoldering" H 4388 4600 30  0001 C CNN
 F 3 "" H 4350 4750 60  0000 C CNN
 	1    4350 4750
@@
 $EndComp
 $Comp
-L C 22pF
+L C 22pF2
 U 1 1 55BF19B7
 P 4350 5050
-F 0 "22pF" H 4375 5150 50  0000 L CNN
+F 0 "22pF2" H 4375 5150 50  0000 L CNN
 F 1 "C2" H 4375 4950 50  0000 L CNN
-F 2 "" H 4388 4900 30  0000 C CNN
+F 2 "Capacitors_SMD:C_0805_HandSoldering" H 4388 4900 30  0001 C CNN
 F 3 "" H 4350 5050 60  0000 C CNN
 	1    4350 5050
@@
 Connection ~ 4700 5050
 $Comp
-L GND #PWR?
+L GND #PWR03
 U 1 1 55BF1A31
 P 4700 5150
-F 0 "#PWR?" H 4700 4900 50  0001 C CNN
+F 0 "#PWR03" H 4700 4900 50  0001 C CNN
 F 1 "GND" H 4700 5000 50  0000 C CNN
 F 2 "" H 4700 5150 60  0000 C CNN
@@
 F 0 "P1" H 3850 6400 50  0000 C CNN
 F 1 "ISP" H 3850 5800 50  0000 C CNN
-F 2 "" H 3850 4900 60  0000 C CNN
+F 2 "Pin_Headers:Pin_Header_Angled_2x05" H 3850 4900 60  0001 C CNN
 F 3 "" H 3850 4900 60  0000 C CNN
 	1    3850 6100
@@
 Connection ~ 4300 6300
 $Comp
-L GND #PWR?
+L GND #PWR04
 U 1 1 55BF20BB
 P 4300 6400
-F 0 "#PWR?" H 4300 6150 50  0001 C CNN
+F 0 "#PWR04" H 4300 6150 50  0001 C CNN
 F 1 "GND" H 4300 6250 50  0000 C CNN
 F 2 "" H 4300 6400 60  0000 C CNN
@@
 	4250 5900 4250 5750
 $Comp
-L VCC #PWR?
+L VCC #PWR05
 U 1 1 55BF2136
 P 4250 5750
-F 0 "#PWR?" H 4250 5600 50  0001 C CNN
+F 0 "#PWR05" H 4250 5600 50  0001 C CNN
 F 1 "VCC" H 4250 5900 50  0000 C CNN
 F 2 "" H 4250 5750 60  0000 C CNN
@@
 LED1
 $Comp
-L USB_B P3
+L USB_B P5
 U 1 1 55BF238B
 P 5750 3850
-F 0 "P3" H 5950 3650 50  0000 C CNN
+F 0 "P5" H 5950 3650 50  0000 C CNN
 F 1 "USB_B" H 5700 4050 50  0000 C CNN
-F 2 "" V 5700 3750 60  0000 C CNN
+F 2 "Connect:USB_A" V 5700 3750 60  0001 C CNN
 F 3 "" V 5700 3750 60  0000 C CNN
 	1    5750 3850
@@
 Connection ~ 5850 4250
 $Comp
-L GND #PWR?
+L GND #PWR06
 U 1 1 55BF2630
 P 5850 4350
-F 0 "#PWR?" H 5850 4100 50  0001 C CNN
+F 0 "#PWR06" H 5850 4100 50  0001 C CNN
 F 1 "GND" H 5850 4200 50  0000 C CNN
 F 2 "" H 5850 4350 60  0000 C CNN
@@
 $EndComp
 $Comp
-L +5V #PWR?
+L +5V #PWR07
 U 1 1 55BF2650
 P 5300 4100
-F 0 "#PWR?" H 5300 3950 50  0001 C CNN
+F 0 "#PWR07" H 5300 3950 50  0001 C CNN
 F 1 "+5V" H 5300 4240 50  0000 C CNN
 F 2 "" H 5300 4100 60  0000 C CNN
@@
 F 0 "R1" V 5630 4700 50  0000 C CNN
 F 1 "68" V 5550 4700 50  0000 C CNN
-F 2 "" V 5480 4700 30  0000 C CNN
+F 2 "Resistors_SMD:R_0805" V 5480 4700 30  0001 C CNN
 F 3 "" H 5550 4700 30  0000 C CNN
 	1    5550 4700
@@
 F 0 "R2" V 5830 4700 50  0000 C CNN
 F 1 "68" V 5750 4700 50  0000 C CNN
-F 2 "" V 5680 4700 30  0000 C CNN
+F 2 "Resistors_SMD:R_0805" V 5680 4700 30  0001 C CNN
 F 3 "" H 5750 4700 30  0000 C CNN
 	1    5750 4700
@@
 F 0 "R5" V 5430 4450 50  0000 C CNN
 F 1 "2K2" V 5350 4450 50  0000 C CNN
-F 2 "" V 5280 4450 30  0000 C CNN
+F 2 "Resistors_SMD:R_0805" V 5280 4450 30  0001 C CNN
 F 3 "" H 5350 4450 30  0000 C CNN
 	1    5350 4450
@@
 Connection ~ 5550 4450
 $Comp
-L ZENERsmall D1
+L ZENERsmall D6
 U 1 1 55BF2D28
 P 6150 4850
-F 0 "D1" H 6150 4950 40  0000 C CNN
+F 0 "D6" H 6150 4950 40  0000 C CNN
 F 1 "ZENERsmall" H 6150 4750 30  0001 C CNN
-F 2 "" H 6150 4850 60  0000 C CNN
+F 2 "Diodes_ThroughHole:Diode_DO-35_SOD27_Horizontal_RM10" H 6150 4850 60  0001 C CNN
 F 3 "" H 6150 4850 60  0000 C CNN
 	1    6150 4850
@@
 $EndComp
 $Comp
-L ZENERsmall D1
+L ZENERsmall D5
 U 1 1 55BF2D5F
 P 6150 5050
-F 0 "D1" H 6150 5150 40  0000 C CNN
+F 0 "D5" H 6150 5150 40  0000 C CNN
 F 1 "ZENERsmall" H 6150 4950 30  0001 C CNN
-F 2 "" H 6150 5050 60  0000 C CNN
+F 2 "Diodes_ThroughHole:Diode_DO-35_SOD27_Horizontal_RM10" H 6150 5050 60  0001 C CNN
 F 3 "" H 6150 5050 60  0000 C CNN
 	1    6150 5050
@@
 Connection ~ 6450 5050
 $Comp
-L GND #PWR?
+L GND #PWR08
 U 1 1 55BF2E93
 P 6450 5150
-F 0 "#PWR?" H 6450 4900 50  0001 C CNN
+F 0 "#PWR08" H 6450 4900 50  0001 C CNN
 F 1 "GND" H 6450 5000 50  0000 C CNN
 F 2 "" H 6450 5150 60  0000 C CNN
@@
 F 0 "U1" H 3800 3500 50  0000 C CNN
 F 1 "AP1117" H 3700 4000 50  0000 C CNN
-F 2 "" H 3700 3750 60  0000 C CNN
+F 2 "SMD_Packages:SOT-223" H 3700 3750 60  0001 C CNN
 F 3 "" H 3700 3750 60  0000 C CNN
 	1    3700 3750
@@
 F 0 "P2" H 4450 3750 50  0000 C CNN
 F 1 "VoltageSelect" V 4550 3550 50  0000 C CNN
-F 2 "" H 4450 3550 60  0000 C CNN
+F 2 "Pin_Headers:Pin_Header_Angled_1x03" H 4450 3550 60  0001 C CNN
 F 3 "" H 4450 3550 60  0000 C CNN
 	1    4450 3550
@@
 	4450 3750 4450 3950
 $Comp
-L VCC #PWR?
+L VCC #PWR09
 U 1 1 55BF3C7B
 P 4450 3950
-F 0 "#PWR?" H 4450 3800 50  0001 C CNN
+F 0 "#PWR09" H 4450 3800 50  0001 C CNN
 F 1 "VCC" H 4450 4100 50  0000 C CNN
 F 2 "" H 4450 3950 60  0000 C CNN
@@
 	4700 3850 4700 3800
 $Comp
-L +5V #PWR?
+L +5V #PWR010
 U 1 1 55BF3DAD
 P 4700 3800
-F 0 "#PWR?" H 4700 3650 50  0001 C CNN
+F 0 "#PWR010" H 4700 3650 50  0001 C CNN
 F 1 "+5V" H 4700 3940 50  0000 C CNN
 F 2 "" H 4700 3800 60  0000 C CNN
@@
 $EndComp
 $Comp
-L +5V #PWR?
+L +5V #PWR011
 U 1 1 55BF3DDB
 P 3400 3750
-F 0 "#PWR?" H 3400 3600 50  0001 C CNN
+F 0 "#PWR011" H 3400 3600 50  0001 C CNN
 F 1 "+5V" H 3400 3890 50  0000 C CNN
 F 2 "" H 3400 3750 60  0000 C CNN
@@
 $EndComp
 $Comp
-L GND #PWR?
+L GND #PWR012
 U 1 1 55BF3E09
 P 3700 4050
-F 0 "#PWR?" H 3700 3800 50  0001 C CNN
+F 0 "#PWR012" H 3700 3800 50  0001 C CNN
 F 1 "GND" H 3700 3900 50  0000 C CNN
 F 2 "" H 3700 4050 60  0000 C CNN
@@
 F 0 "D3" H 5400 7050 50  0000 C CNN
 F 1 "LED_GREEN" H 5400 6850 50  0000 C CNN
-F 2 "" H 5400 6950 60  0000 C CNN
+F 2 "LEDs:LED-5MM" H 5400 6950 60  0001 C CNN
 F 3 "" H 5400 6950 60  0000 C CNN
 	1    5400 6950
@@
 F 0 "D4" H 5800 7050 50  0000 C CNN
 F 1 "LED_RED" H 5800 6850 50  0000 C CNN
-F 2 "" H 5800 6950 60  0000 C CNN
+F 2 "LEDs:LED-5MM" H 5800 6950 60  0001 C CNN
 F 3 "" H 5800 6950 60  0000 C CNN
 	1    5800 6950
@@
 F 0 "R9" V 5480 6450 50  0000 C CNN
 F 1 "1K" V 5400 6450 50  0000 C CNN
-F 2 "" V 5330 6450 30  0000 C CNN
+F 2 "Resistors_SMD:R_0805" V 5330 6450 30  0001 C CNN
 F 3 "" H 5400 6450 30  0000 C CNN
 	1    5400 6450
@@
 F 0 "R10" V 5880 6450 50  0000 C CNN
 F 1 "1K" V 5800 6450 50  0000 C CNN
-F 2 "" V 5730 6450 30  0000 C CNN
+F 2 "Resistors_SMD:R_0805" V 5730 6450 30  0001 C CNN
 F 3 "" H 5800 6450 30  0000 C CNN
 	1    5800 6450
@@
 	5800 7400 5300 7400
 $Comp
-L +5V #PWR?
+L +5V #PWR013
 U 1 1 55BF5166
 P 5400 6100
-F 0 "#PWR?" H 5400 5950 50  0001 C CNN
+F 0 "#PWR013" H 5400 5950 50  0001 C CNN
 F 1 "+5V" H 5400 6240 50  0000 C CNN
 F 2 "" H 5400 6100 60  0000 C CNN
@@
 $EndComp
 $Comp
-L +5V #PWR?
+L +5V #PWR014
 U 1 1 55BF51D9
 P 5800 6100
-F 0 "#PWR?" H 5800 5950 50  0001 C CNN
+F 0 "#PWR014" H 5800 5950 50  0001 C CNN
 F 1 "+5V" H 5800 6240 50  0000 C CNN
 F 2 "" H 5800 6100 60  0000 C CNN
@@
 F 0 "P3" H 3850 7200 50  0000 C CNN
 F 1 "SlowCLK" V 3950 7050 50  0000 C CNN
-F 2 "" H 3850 7050 60  0000 C CNN
+F 2 "Pin_Headers:Pin_Header_Angled_1x02" H 3850 7050 60  0001 C CNN
 F 3 "" H 3850 7050 60  0000 C CNN
 	1    3850 7050
@@
 $EndComp
 $Comp
-L CONN_01X02 P2
+L CONN_01X02 P4
 U 1 1 55BF5BDD
 P 4550 7050
-F 0 "P2" H 4550 7200 50  0000 C CNN
+F 0 "P4" H 4550 7200 50  0000 C CNN
 F 1 "SelfPrograming" V 4650 7050 50  0000 C CNN
-F 2 "" H 4550 7050 60  0000 C CNN
+F 2 "Pin_Headers:Pin_Header_Angled_1x02" H 4550 7050 60  0001 C CNN
 F 3 "" H 4550 7050 60  0000 C CNN
 	1    4550 7050
@@
 F 0 "R8" V 2930 6900 50  0000 C CNN
 F 1 "1K" V 2850 6900 50  0000 C CNN
-F 2 "" V 2780 6900 30  0000 C CNN
+F 2 "Resistors_SMD:R_0805_HandSoldering" V 2780 6900 30  0001 C CNN
 F 3 "" H 2850 6900 30  0000 C CNN
 	1    2850 6900
@@
 F 0 "R11" V 3080 6400 50  0000 C CNN
 F 1 "1K" V 3000 6400 50  0000 C CNN
-F 2 "" V 2930 6400 30  0000 C CNN
+F 2 "Resistors_SMD:R_0805_HandSoldering" V 2930 6400 30  0001 C CNN
 F 3 "" H 3000 6400 30  0000 C CNN
 	1    3000 6400
@@
 $EndComp
 $Comp
-L VCC #PWR?
+L VCC #PWR015
 U 1 1 55BF7D24
 P 3000 6250
-F 0 "#PWR?" H 3000 6100 50  0001 C CNN
+F 0 "#PWR015" H 3000 6100 50  0001 C CNN
 F 1 "VCC" H 3000 6400 50  0000 C CNN
 F 2 "" H 3000 6250 60  0000 C CNN
@@
 	3000 6650 3000 6550
 $Comp
-L GND #PWR?
+L GND #PWR016
 U 1 1 55BFB054
 P 3550 7300
-F 0 "#PWR?" H 3550 7050 50  0001 C CNN
+F 0 "#PWR016" H 3550 7050 50  0001 C CNN
 F 1 "GND" H 3550 7150 50  0000 C CNN
 F 2 "" H 3550 7300 60  0000 C CNN

Commit message: Plotter specific PCB added
Parts:
- removed R8: 1K, Resistors_SMD:R_0805_HandSoldering, symbol R
Connections:
- net RXD: no longer names the net of IC1.30 ((PCINT16/RXD)PD0)
- net RXD: no longer P1.6 (P6)
- net TXD: no longer names the net of P1.4 (P4)
Changed lines of the file:
@@
 Text GLabel 2650 5500 2    39   Input ~ 0
 MOSI
-Text GLabel 2650 6800 2    39   Input ~ 0
-RXD
-Text GLabel 3100 6900 2    39   Input ~ 0
-TXD
 $Comp
 L VCC #PWR01
@@
 Text GLabel 3600 6300 0    39   Input ~ 0
 MISO
-Text GLabel 4100 6000 2    39   Input ~ 0
-TXD
-Text GLabel 4100 6100 2    39   Input ~ 0
-RXD
 Wire Wire Line
 	4100 6200 4300 6200
@@
 RST_SS
 $Comp
-L R R8
-U 1 1 55BF68E1
-P 2850 6900
-F 0 "R8" V 2930 6900 50  0000 C CNN
-F 1 "1K" V 2850 6900 50  0000 C CNN
-F 2 "Resistors_SMD:R_0805_HandSoldering" V 2780 6900 30  0001 C CNN
-F 3 "" H 2850 6900 30  0000 C CNN
-	1    2850 6900
-	0    1    1    0
-$EndComp
-Wire Wire Line
-	2700 6900 2650 6900
-Wire Wire Line
-	3000 6900 3100 6900
-$Comp
 L R R11
